Commit message: Why did libfranka fix every name of the link?

File: urdf/panda_modified.urdf (robot description, URDF)
Before this commit: robot panda, 13 links, 12 joints
Links:
- removed link panda_grasptarget
- removed link panda_hand
- removed link panda_leftfinger
- removed link panda_link0
- removed link panda_link1
- removed link panda_link2
- removed link panda_link3
- removed link panda_link4
- removed link panda_link5
- removed link panda_link6
- removed link panda_link7
- removed link panda_link8
- removed link panda_rightfinger
- added link link0, mass 2.9; collision mesh filename=package://meshes/collision/link0.obj; visual mesh filename=package://meshes/collision/link0.obj
- added link link1, mass 2.7; collision mesh filename=package://meshes/collision/link1.obj; visual mesh filename=package://meshes/visual/link1.obj
- added link link2, mass 2.73; collision mesh filename=package://meshes/collision/link2.obj; visual mesh filename=package://meshes/visual/link2.obj
- added link link3, mass 2.04; collision mesh filename=package://meshes/collision/link3.obj; visual mesh filename=package://meshes/visual/link3.obj
- added link link4, mass 2.08; collision mesh filename=package://meshes/collision/link4.obj; visual mesh filename=package://meshes/visual/link4.obj
- added link link5, mass 3; collision mesh filename=package://meshes/collision/link5.obj; visual mesh filename=package://meshes/visual/link5.obj
- added link link6, mass 1.3; collision mesh filename=package://meshes/collision/link6.obj; visual mesh filename=package://meshes/visual/link6.obj
- added link link7, mass .2; collision mesh filename=package://meshes/collision/link7.obj; visual mesh filename=package://meshes/collision/link7.obj
- added link link8, mass 0.0
Joints:
- removed joint panda_finger_joint1
- removed joint panda_finger_joint2
- removed joint panda_grasptarget_hand
- removed joint panda_hand_joint
- joint joint1: child panda_link1 -> link1; parent panda_link0 -> link0
- joint joint2: child panda_link2 -> link2; parent panda_link1 -> link1
- joint joint3: child panda_link3 -> link3; parent panda_link2 -> link2
- joint joint4: child panda_link4 -> link4; parent panda_link3 -> link3
- joint joint5: child panda_link5 -> link5; parent panda_link4 -> link4
- joint joint6: child panda_link6 -> link6; parent panda_link5 -> link5
- joint joint7: child panda_link7 -> link7; parent panda_link6 -> link6
- joint panda_joint8: child panda_link8 -> link8; parent panda_link7 -> link7
